File: embedded/Breath_mask/Breath_mask.kicad_sch (KiCad schematic)
At the start: 27 parts, among them IC1 TPS61291DRVR, J1 Conn_01x02_Pin, J2 USB, J4 Conn_ST_STDC14, SW2 SW_Push, SW3 SW_Push, U1 LPS22HBTR, U23 M95256, U4 STM32L052K8Tx

Commit message: setup schematic
Parts:
- added R1, R2: 22, symbol Device:R
- added R3, R4: 5.1k, symbol Device:R
- added R5: 100k, symbol Device:R
- added R6: 150k, symbol Device:R
Connections:
- net GND: now also R3.2, R4.2, R6.1
- net USB_DM: now also J2.A7 (D-), J2.B7 (D-), R1.2; no longer U4.21 (PA11)
- net USB_DP: now also J2.A6 (D+), J2.B6 (D+), R2.2; no longer U4.22 (PA12)
- net USB_F: now reaches U4.8 (PA2)
- net USB_F: now also R5.2, R6.2
- net at J2.A4 (VBUS), J2.A9 (VBUS), J2.B4 (VBUS)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: now also R5.1
- net at J2.A5 (CC1): now also R4.1
- net at J2.B5 (CC2): now also R3.1
- new net: R1.1, U4.21 (PA11)
- new net: R2.1, U4.22 (PA12)
- no-connect marks 5 -> 7
Other:
- moved on the sheet: J2

Commit message: inizio sbroglio pcb
Parts:
- removed J1: Conn_01x02_Pin, symbol Connector:Conn_01x02_Pin
- removed RN21: 33, Resistor_SMD:R_Array_Convex_4x0603, symbol Device:R_Pack04
- added R12, R13, R14, R15: 33, Resistor_SMD:R_0603_1608Metric, symbol Device:R
- added TP1, TP2, TP3: TestPoint, TestPoint:TestPoint_Pad_D1.0mm, symbol Connector:TestPoint
- BT1: footprint (none) -> Battery:BatteryHolder_Keystone_3034_1x20mm
- C1, C2, C4, C5, C8: footprint (none) -> Capacitor_SMD:C_0603_1608Metric
- C10, C3, C6, C9: footprint (none) -> Capacitor_SMD:C_0805_2012Metric
- IC1: footprint SON65P200X200X80-7N -> Package_SON:WSON-6-1EP_2x2mm_P0.65mm_EP1x1.6mm_ThermalVias
- J4: footprint eagle_connectors:SAMTEC_FTSH-107-01-L-DV-K-TR -> impronte_breath_mask:SAMTEC_FTSH-107-01-L-DV-K-TR
- L1: footprint (none) -> Inductor_SMD:L_Coilcraft_LPS3314
- R1, R2, R3, R4, R5, R6, R7: footprint (none) -> Resistor_SMD:R_0603_1608Metric
- SW2: footprint (none) -> Button_Switch_SMD:SW_SPDT_CK_JS102011SAQN
- SW3: footprint (none) -> Button_Switch_SMD:SW_Push_1P1T_XKB_TS-1187A
Connections:
- net +3V3: now also TP1.1
- net GND: now also TP3.1
- net MEM_CS: now also R15.2; no longer U4.10 (PA4)
- net SPI1_MISO: now also U23.2 (Q), R13.1; no longer U4.12 (PA6)
- net SPI1_MOSI: now also U23.5 (D), R14.2; no longer U4.13 (PA7)
- net SPI1_SCK: now also U23.6 (C), R12.2; no longer U4.11 (PA5)
- net at BT1.1 (+), SW2.1: now also TP2.1
- new net: R15.1, U4.10 (PA4)
- new net: R12.1, U4.11 (PA5)
- new net: R13.2, U4.12 (PA6)
- new net: R14.1, U4.13 (PA7)
- no-connect marks 7 -> 17
Other:
- note added: "Micro"
- note added: "Power supply 3V -> 3.3V"
- note added: "Pressure Sensor"
- note added: "UART Connector"
- note added: "USB-C"
- moved on the sheet: C1, C10, C11, C2, C3, C4, C5, C6, C8, C9, IC1, J2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

Commit message: errors fixed
Connections:
- net ~{HOLD}: now also U4.2 (PC14)
- net ~{W}: now also U4.3 (PC15)
- no-connect marks 17 -> 15
Changed lines of the file:
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@@
-	)
-	(no_connect
-		(at 201.93 148.59)
 	)
 	(no_connect
@@
 	)
 	(no_connect
-		(at 201.93 146.05)
-	)
-	(no_connect
 		(at 201.93 158.75)
 	)
@@
 		)
 	)
+	(wire
+		(pts
+			(xy 190.5 148.59) (xy 201.93 148.59)
+		)
+		(stroke
+			(width 0)
+			(type default)
+		)
+	)
 	(polyline
 		(pts
@@
 		(pts
 			(xy 185.42 63.5) (xy 185.42 66.04)
+		)
+		(stroke
+			(width 0)
+			(type default)
+		)
+	)
+	(wire
+		(pts
+			(xy 190.5 146.05) (xy 201.93 146.05)
 		)
 		(stroke
@@
 		)
 	)
+	(label "~{HOLD}"
+		(at 190.5 146.05 0)
+		(effects
+			(font
+				(size 1.27 1.27)
+			)
+			(justify left bottom)
+		)
+	)
 	(label "USB_F"
 		(at 259.08 135.89 180)
@@
 		(effects
 			(font
+				(size 1.27 1.27)
+			)
+			(justify left bottom)
+		)
+	)
+	(label "~{W}"
+		(at 190.5 148.59 0)
+		(effects
+			(font

Commit message: firmware: initialized
Parts:
- U4: LCSC (none) -> C222404
Changed lines of the file:
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@@
+			)
+		)
+		(property "LCSC" "C222404"
+			(at 217.17 156.21 0)
+			(hide yes)
+			(show_name no)
+			(do_not_autoplace no)
+			(effects
+				(font
+					(size 1.27 1.27)
+				)
 			)
 		)
